Commit message: 修改urdf文件中mesh路径为相对路径

File: source/robot_lab/data/Robots/unitree/Go2Arm_description/urdf/go2_piper_description_mjc.urdf (robot description, URDF)
Before this commit: robot go2_description, 52 links, 51 joints
Links:
- link FL_calf: geometry collision cylinder length=0.12 radius=0.012; visual mesh filename=../meshes/calf.stl
- link FL_foot: geometry collision sphere radius=0.022; visual mesh filename=../meshes/foot.stl
- link FL_hip: geometry collision cylinder length=0.04 radius=0.046; visual mesh filename=../meshes/hip.stl
- link FL_thigh: geometry collision box size=0.213 0.0245 0.034; visual mesh filename=../meshes/thigh.stl
- link FR_calf: geometry collision cylinder length=0.12 radius=0.013; visual mesh filename=../meshes/calf_mirror.stl
- link FR_foot: geometry collision sphere radius=0.022; visual mesh filename=../meshes/foot.stl
- link FR_hip: geometry collision cylinder length=0.04 radius=0.046; visual mesh filename=../meshes/hip.stl
- link FR_thigh: geometry collision box size=0.213 0.0245 0.034; visual mesh filename=../meshes/thigh_mirror.stl
- link RL_calf: geometry collision cylinder length=0.12 radius=0.013; visual mesh filename=../meshes/calf.stl
- link RL_foot: geometry collision sphere radius=0.022; visual mesh filename=../meshes/foot.stl
- link RL_hip: geometry collision cylinder length=0.04 radius=0.046; visual mesh filename=../meshes/hip.stl
- link RL_thigh: geometry collision box size=0.213 0.0245 0.034; visual mesh filename=../meshes/thigh.stl
- link RR_calf: geometry collision cylinder length=0.12 radius=0.013; visual mesh filename=../meshes/calf_mirror.stl
- link RR_foot: geometry collision sphere radius=0.022; visual mesh filename=../meshes/foot.stl
- link RR_hip: geometry collision cylinder length=0.04 radius=0.046; visual mesh filename=../meshes/hip.stl
- link RR_thigh: geometry collision box size=0.213 0.0245 0.034; visual mesh filename=../meshes/thigh_mirror.stl
- link base: geometry collision box size=0.3762 0.0935 0.114; visual mesh filename=../meshes/base.stl
- link base_link: geometry collision mesh filename=../meshes/base_link.STL; visual mesh filename=../meshes/base_link.STL
- link gripper_base: geometry collision mesh filename=../meshes/gripper_base.STL; visual mesh filename=../meshes/gripper_base.STL
- link link1: geometry collision mesh filename=../meshes/link1.STL; visual mesh filename=../meshes/link1.STL
- link link2: geometry collision mesh filename=../meshes/link2.STL; visual mesh filename=../meshes/link2.STL
- link link3: geometry collision mesh filename=../meshes/link3.STL; visual mesh filename=../meshes/link3.STL
- link link4: geometry collision mesh filename=../meshes/link4.STL; visual mesh filename=../meshes/link4.STL
- link link5: geometry collision mesh filename=../meshes/link5.STL; visual mesh filename=../meshes/link5.STL
- link link6: geometry collision mesh filename=../meshes/link6.STL; visual mesh filename=../meshes/link6.STL
- link link7: geometry collision mesh filename=../meshes/link7.STL; visual mesh filename=../meshes/link7.STL
- link link8: geometry collision mesh filename=../meshes/link8.STL; visual mesh filename=../meshes/link8.STL
