Commit message: 已改为能跑训练的版本，还差curriculum和teacher-student部分的修改

File: source/robot_lab/data/Robots/unitree/Go2Arm_description/urdf/go2_piper_description_mjc_NoGripper.urdf (robot description, URDF)
Before this commit: robot go2_description, 50 links, 49 joints
Links:
- removed link gripper_base
Joints:
- removed joint joint6_to_gripper_base
